Commit message: fixing wheels

File: summit_xl_description/urdf/bases/summit_xl_base.urdf.xacro (robot description, xacro)
@@ -35,5 +35,6 @@
         <origin xyz="0 0 0" rpy="0 0 0 " />
         <geometry>
-          <mesh filename="file://$(find summit_xl_description)/meshes/bases/summit_xl_chassis_collision.dae"/>
+          <!-- <mesh filename="file://$(find summit_xl_description)/meshes/bases/summit_xl_chassis_collision.dae"/> -->
+          <box size="0.01 0.01 0.01" />
         </geometry>
       </collision>

File: summit_xl_description/urdf/wheels/rubber_wheel.urdf.xacro (robot description, xacro)
@@ -15,6 +15,6 @@
       <child link="${prefix}wheel_link"/>
       <axis xyz="0 1 0" rpy="0 0 0" />
-      <limit effort="100" velocity="100"/>
-      <dynamics damping="0.05" friction="0.1"/>
+      <limit effort="1000" velocity="10"/>
+      <dynamics damping="0.05" friction="0.01"/>
     </joint>
     <link name="${prefix}wheel_link">
@@ -53,10 +53,9 @@
     </link>
     <gazebo reference="${prefix}wheel_link">
-      <mu1>0.95</mu1>
-      <mu2>0.90</mu2>
-      <kp>2.75e6</kp>
-      <kd>8.25e1</kd>
-      <fdir1>0 0 0</fdir1>
-      <maxContacts>4</maxContacts>
+      <mu1>1.0</mu1>
+      <mu2>0.5</mu2>
+      <kp>10000000</kp>
+      <kd>1.0</kd>
+      <fdir1>0 1 0</fdir1>
     </gazebo>
   </xacro:macro>
