Commit message: fixing summit_xl_std

File: summit_xl_description/robots/summit_xl_std.urdf.xacro (robot description, xacro)
@@ -4,5 +4,5 @@
   <!-- Imported elements -->
   <!-- ***************** -->
-  <!-- Import RB1 base elements (base + wheels) -->
+  <!-- Import summit base elements (base + wheels) -->
   <xacro:include filename="$(find summit_xl_description)/urdf/bases/summit_xl_base.urdf.xacro"/>
   <xacro:include filename="$(find summit_xl_description)/urdf/wheels/rubber_wheel.urdf.xacro"/>
@@ -30,45 +30,48 @@
   <!-- *************** -->
   <!-- Summit XL -->
-  <xacro:summit_xl_base prefix="$(arg prefix)" publish_bf="true" hq="${hq}"/>
+  <xacro:summit_xl_base prefix="$(arg prefix)/" publish_bf="true" hq="${hq}"/>
   <!--xacro:gazebo_colors /-->
   <!-- WHEELS -->
   <xacro:unless value="$(arg omni_wheels)">
-    <xacro:rubber_wheel prefix="front_right_" parent="$(arg prefix)base_link" reflect="false" hq="${hq}">
+    <xacro:rubber_wheel prefix="front_right_" parent="$(arg prefix)/base_link" reflect="false" hq="${hq}">
       <origin xyz="${wheel_offset_x} -${wheel_offset_y} ${wheel_offset_z}" rpy="0 0 0"/>
     </xacro:rubber_wheel>
-    <xacro:rubber_wheel prefix="front_left_" parent="$(arg prefix)base_link" reflect="true" hq="${hq}">
+    <xacro:rubber_wheel prefix="front_left_" parent="$(arg prefix)/base_link" reflect="true" hq="${hq}">
       <origin xyz="${wheel_offset_x} ${wheel_offset_y} ${wheel_offset_z}" rpy="0 0 0"/>
     </xacro:rubber_wheel>
-    <xacro:rubber_wheel prefix="rear_left_" parent="$(arg prefix)base_link" reflect="true" hq="${hq}">
+    <xacro:rubber_wheel prefix="rear_left_" parent="$(arg prefix)/base_link" reflect="true" hq="${hq}">
       <origin xyz="-${wheel_offset_x} ${wheel_offset_y} ${wheel_offset_z}" rpy="0 0 0"/>
     </xacro:rubber_wheel>
-    <xacro:rubber_wheel prefix="rear_right_" parent="$(arg prefix)base_link" reflect="false" hq="${hq}">
+    <xacro:rubber_wheel prefix="rear_right_" parent="$(arg prefix)/base_link" reflect="false" hq="${hq}">
       <origin xyz="-${wheel_offset_x} -${wheel_offset_y} ${wheel_offset_z}" rpy="0 0 0"/>
     </xacro:rubber_wheel>
   </xacro:unless>
   <xacro:if value="$(arg omni_wheels)">
-    <xacro:omni_wheel prefix="front_right_" parent="$(arg prefix)base_link" reflect="false" hq="${hq}">
+    <xacro:omni_wheel prefix="front_right_" parent="$(arg prefix)/base_link" reflect="false" hq="${hq}">
       <origin xyz="${wheel_offset_x} -${wheel_offset_y} ${wheel_offset_z}" rpy="0 0 0"/>
     </xacro:omni_wheel>
-    <xacro:omni_wheel prefix="front_left_" parent="$(arg prefix)base_link" reflect="true" hq="${hq}">
+    <xacro:omni_wheel prefix="front_left_" parent="$(arg prefix)/base_link" reflect="true" hq="${hq}">
       <origin xyz="${wheel_offset_x} ${wheel_offset_y} ${wheel_offset_z}" rpy="0 0 0"/>
     </xacro:omni_wheel>
-    <xacro:omni_wheel prefix="back_left_" parent="$(arg prefix)base_link" reflect="true" hq="${hq}">
+    <xacro:omni_wheel prefix="back_left_" parent="$(arg prefix)/base_link" reflect="true" hq="${hq}">
       <origin xyz="-${wheel_offset_x} ${wheel_offset_y} ${wheel_offset_z}" rpy="0 0 0"/>
     </xacro:omni_wheel>
-    <xacro:omni_wheel prefix="back_right_" parent="$(arg prefix)base_link" reflect="false" hq="${hq}">
+    <xacro:omni_wheel prefix="back_right_" parent="$(arg prefix)/base_link" reflect="false" hq="${hq}">
       <origin xyz="-${wheel_offset_x} -${wheel_offset_y} ${wheel_offset_z}" rpy="0 0 0"/>
     </xacro:omni_wheel>
   </xacro:if>
   <!-- SENSORS -->
-  <xacro:sensor_robosense_helios node_namespace="$(arg robot_ns)" frame_prefix="$(arg prefix)front_laser_" parent="$(arg prefix)base_link">
-      <origin xyz="-0.11808 0.0 0.38509" rpy="0 0 0"/>
-  </xacro:sensor_robosense_helios>
-  <xacro:sensor_stereolabs_zed2 node_namespace="$(arg robot_ns)" frame_prefix="$(arg prefix)front_camera_" parent="$(arg prefix)base_link">
+  <xacro:sensor_robosense_helios_16p simulation="true" gpu="true" node_namespace="$(arg robot_ns)" frame_prefix="$(arg prefix)/front_laser_" parent="$(arg prefix)/base_link">
+      <origin xyz="0.0 0.0 0.275" rpy="0 0 0"/>
+  </xacro:sensor_robosense_helios_16p>
+  <xacro:sensor_stereolabs_zed2 simulation="true" node_namespace="$(arg robot_ns)" node_name="zed2" frame_prefix="$(arg prefix)/front_camera_" parent="$(arg prefix)/base_link">
       <origin xyz="0.324 0.012 0.172" rpy="0 0 0"/>
   </xacro:sensor_stereolabs_zed2>
-  <xacro:structure_mastil_gps prefix="$(arg prefix)gps" parent="$(arg prefix)base_link">
-    <origin xyz="-0.24 0.095 0.30" rpy="0 0 0"/>
+  <xacro:structure_mastil_gps prefix="$(arg prefix)/gps" parent="$(arg prefix)/base_link">
+    <origin xyz="-0.24 0.095 0.275" rpy="0 0 0"/>
   </xacro:structure_mastil_gps>
+	<xacro:sensor_ublox simulation="true" frame_prefix="$(arg prefix)/gps/" node_namespace="$(arg robot_ns)" topic_prefix="gps/" parent="$(arg prefix)/gps_link">
+	  <origin xyz="0.0 0 0.37" rpy="0 0 0"/>
+	</xacro:sensor_ublox>
   <!-- Gazebo ros control plugins -->
   <xacro:arg name="config_controllers" default=""/>

File: summit_xl_description/urdf/ros2_control.urdf.xacro (robot description, xacro)
@@ -4,6 +4,9 @@
       <gazebo>
         <plugin name="ros_control" filename="libgazebo_ros2_control.so">
-          <namespace>$(arg robot_id)</namespace>
           <parameters>$(arg config_controllers)</parameters>
+          <ros>
+            <namespace>$(arg robot_id)</namespace>
+            <remapping>~/cmd_vel_unstamped:=~/cmd_vel</remapping>
+          </ros>
         </plugin>
       </gazebo>

Commit message: adding imu to summit

File: summit_xl_description/robots/summit_xl_std.urdf.xacro (robot description, xacro)
@@ -74,4 +74,7 @@
 	  <origin xyz="0.0 0 0.37" rpy="0 0 0"/>
 	</xacro:sensor_ublox>
+	<xacro:sensor_myahrs simulation="true" frame_prefix="$(arg prefix)/imu/" node_namespace="$(arg robot_ns)" parent="$(arg prefix)/base_link">
+		<origin xyz="0.127 -0.129 0.212" rpy="0 0 0"/>
+  </xacro:sensor_myahrs>
   <!-- Gazebo ros control plugins -->
   <xacro:arg name="config_controllers" default=""/>

Commit message: new sensor structures

File: summit_xl_description/robots/summit_xl_std.urdf.xacro (robot description, xacro)
@@ -9,4 +9,6 @@
   <xacro:include filename="$(find summit_xl_description)/urdf/wheels/omni_wheel.urdf.xacro"/>
   <xacro:include filename="$(find summit_xl_description)/urdf/structures/structure_gps.urdf.xacro"/>
+  <xacro:include filename="$(find summit_xl_description)/urdf/structures/structure_robosense.urdf.xacro"/>
+  <xacro:include filename="$(find summit_xl_description)/urdf/structures/structure_teltonika.urdf.xacro"/>
   <!-- Import all available sensors -->
   <xacro:include filename="$(find robotnik_sensors)/urdf/all_sensors.urdf.xacro"/>
@@ -62,18 +64,29 @@
   </xacro:if>
   <!-- SENSORS -->
-  <xacro:sensor_robosense_helios_16p simulation="true" gpu="true" node_namespace="$(arg robot_ns)" frame_prefix="$(arg prefix)/front_laser_" parent="$(arg prefix)/base_link">
-      <origin xyz="0.0 0.0 0.275" rpy="0 0 0"/>
+  <!-- 3D Lidar-->
+  <xacro:structure_robosense prefix="$(arg prefix)/front_laser_" parent="$(arg prefix)/base_link">
+    <origin xyz="-0.11924 0.0 0.32069" rpy="0 0 0"/>
+  </xacro:structure_robosense>
+  <xacro:sensor_robosense_helios_16p simulation="true" gpu="true" node_namespace="$(arg robot_ns)" frame_prefix="$(arg prefix)/front_laser_" parent="$(arg prefix)/front_laser_structure_robosense">
+    <origin xyz="0.0 0.0 0.04569" rpy="0 0 0"/>
   </xacro:sensor_robosense_helios_16p>
-  <xacro:sensor_stereolabs_zed2i_low_res simulation="true" node_namespace="$(arg robot_ns)" node_name="zed2" frame_prefix="$(arg prefix)/front_camera_" parent="$(arg prefix)/base_link">
-      <origin xyz="0.324 0.012 0.172" rpy="0 0 0"/>
-  </xacro:sensor_stereolabs_zed2i_low_res>
+  <!-- CAMERA -->
+  <xacro:sensor_stereolabs_zed2_low_res simulation="true" node_namespace="$(arg robot_ns)" node_name="zed2" frame_prefix="$(arg prefix)/front_camera_" parent="$(arg prefix)/base_link">
+    <origin xyz="0.324 0.012 0.172" rpy="0 0 0"/>
+  </xacro:sensor_stereolabs_zed2_low_res>
+  <!-- GPS -->
   <xacro:structure_mastil_gps prefix="$(arg prefix)/gps" parent="$(arg prefix)/base_link">
-    <origin xyz="-0.24 0.095 0.275" rpy="0 0 0"/>
+    <origin xyz="-0.24824 0.095 0.275" rpy="0 0 0"/>
   </xacro:structure_mastil_gps>
-	<xacro:sensor_ublox simulation="true" frame_prefix="$(arg prefix)/gps/" node_namespace="$(arg robot_ns)" topic_prefix="gps/" parent="$(arg prefix)/gps_link">
-	  <origin xyz="0.0 0 0.37" rpy="0 0 0"/>
-	</xacro:sensor_ublox>
-	<xacro:sensor_myahrs simulation="true" frame_prefix="$(arg prefix)/imu/" node_namespace="$(arg robot_ns)" parent="$(arg prefix)/base_link">
-		<origin xyz="0.127 -0.129 0.212" rpy="0 0 0"/>
+  <xacro:sensor_ublox simulation="true" frame_prefix="$(arg prefix)/gps/" node_namespace="$(arg robot_ns)" topic_prefix="gps/" parent="$(arg prefix)/gps_link">
+    <origin xyz="0.0 0 0.37" rpy="0 0 0"/>
+  </xacro:sensor_ublox>
+  <!-- Antenna -->
+  <xacro:structure_mastil_teltonika prefix="$(arg prefix)/antenna" parent="$(arg prefix)/base_link">
+    <origin xyz="-0.24824 -0.095 0.275" rpy="0 0 0"/>
+  </xacro:structure_mastil_teltonika>
+  <!-- IMU -->
+  <xacro:sensor_myahrs simulation="true" frame_prefix="$(arg prefix)/imu/" node_namespace="$(arg robot_ns)" parent="$(arg prefix)/base_link">
+    <origin xyz="0.03534 0.132 0.14138" rpy="0 0 0"/>
   </xacro:sensor_myahrs>
   <!-- Gazebo ros control plugins -->

Commit message: adding asus xtion

File: summit_xl_description/robots/summit_xl_std.urdf.xacro (robot description, xacro)
@@ -13,4 +13,5 @@
   <!-- Import all available sensors -->
   <xacro:include filename="$(find robotnik_sensors)/urdf/all_sensors.urdf.xacro"/>
+  <xacro:include filename="$(find asus_xtion_description)/urdf/asus_xtion.urdf.xacro"/>
   <!-- ***************** -->
   <!-- Global parameters -->
@@ -75,4 +76,26 @@
     <origin xyz="0.324 0.012 0.172" rpy="0 0 0"/>
   </xacro:sensor_stereolabs_zed2i_low_res>
+  <link name="$(arg prefix)/camera_mast_link">
+    <visual>
+      <origin rpy="0 0 0" xyz="0 0 0" />
+      <geometry>
+        <box size="0.025 0.025 1.2"/>
+      </geometry>
+    </visual>
+    <collision>
+      <origin rpy="0 0 0" xyz="0 0 0" />
+      <geometry>
+        <box size="0.025 0.025 1.2"/>
+      </geometry>
+    </collision>
+  </link>
+  <joint name="$(arg prefix)/camera_mast_link_joint" type="fixed">
+    <origin rpy="0 0 0" xyz="-0.26 0.0 0.875"/>
+    <parent link="$(arg prefix)/base_link" />
+    <child link="$(arg prefix)/camera_mast_link" />
+  </joint>
+  <xacro:sensor_asus_xtion parent="$(arg prefix)/camera_mast_link" name="camera">
+    <origin xyz="0.045 0.0 0.57" rpy="0 ${pi/5} 0"/>
+  </xacro:sensor_asus_xtion>
   <!-- GPS -->
   <xacro:structure_mastil_gps prefix="$(arg prefix)/gps" parent="$(arg prefix)/base_link">

Commit message: fixing asus positions

File: summit_xl_description/robots/summit_xl_std.urdf.xacro (robot description, xacro)
@@ -80,5 +80,5 @@
       <origin rpy="0 0 0" xyz="0 0 0" />
       <geometry>
-        <box size="0.025 0.025 1.2"/>
+        <box size="0.03 0.03 1.2"/>
       </geometry>
     </visual>
@@ -86,5 +86,5 @@
       <origin rpy="0 0 0" xyz="0 0 0" />
       <geometry>
-        <box size="0.025 0.025 1.2"/>
+        <box size="0.03 0.03 1.2"/>
       </geometry>
     </collision>

Commit message: moving asus camera to the front

File: summit_xl_description/robots/summit_xl_std.urdf.xacro (robot description, xacro)
@@ -80,5 +80,5 @@
       <origin rpy="0 0 0" xyz="0 0 0" />
       <geometry>
-        <box size="0.03 0.03 1.2"/>
+        <box size="0.02 0.02 0.5"/>
       </geometry>
     </visual>
@@ -86,15 +86,15 @@
       <origin rpy="0 0 0" xyz="0 0 0" />
       <geometry>
-        <box size="0.03 0.03 1.2"/>
+        <box size="0.02 0.02 0.5"/>
       </geometry>
     </collision>
   </link>
   <joint name="$(arg prefix)/camera_mast_link_joint" type="fixed">
-    <origin rpy="0 0 0" xyz="-0.26 0.0 0.875"/>
+    <origin rpy="0 0 0" xyz="0.025 0.0 0.525"/>
     <parent link="$(arg prefix)/base_link" />
     <child link="$(arg prefix)/camera_mast_link" />
   </joint>
   <xacro:sensor_asus_xtion parent="$(arg prefix)/camera_mast_link" name="camera">
-    <origin xyz="0.045 0.0 0.57" rpy="0 ${pi/5} 0"/>
+    <origin xyz="0.04 0.0 0.243" rpy="0 ${pi/5} 0"/>
   </xacro:sensor_asus_xtion>
   <!-- GPS -->

Commit message: adding realsense d455

File: summit_xl_description/robots/summit_xl_std.urdf.xacro (robot description, xacro)
@@ -13,5 +13,5 @@
   <!-- Import all available sensors -->
   <xacro:include filename="$(find robotnik_sensors)/urdf/all_sensors.urdf.xacro"/>
-  <xacro:include filename="$(find asus_xtion_description)/urdf/asus_xtion.urdf.xacro"/>
+  <xacro:include filename="$(find realsense2_description)/urdf/_d455.urdf.xacro" />
   <!-- ***************** -->
   <!-- Global parameters -->
@@ -90,12 +90,31 @@
     </collision>
   </link>
-  <joint name="$(arg prefix)/camera_mast_link_joint" type="fixed">
+  <joint name="$(arg prefix)/camera_mast_joint" type="fixed">
     <origin rpy="0 0 0" xyz="0.025 0.0 0.525"/>
     <parent link="$(arg prefix)/base_link" />
     <child link="$(arg prefix)/camera_mast_link" />
   </joint>
-  <xacro:sensor_asus_xtion parent="$(arg prefix)/camera_mast_link" name="camera">
-    <origin xyz="0.04 0.0 0.243" rpy="0 ${pi/5} 0"/>
-  </xacro:sensor_asus_xtion>
+  <link name="$(arg prefix)/d455_base_link">
+    <visual>
+      <origin xyz="0 0 0" rpy="0 0 0"/>
+      <geometry>
+        <mesh filename="file://$(find summit_xl_description)/meshes/structures/d455_base.stl" scale="0.001 0.001 0.001"/>
+      </geometry>
+    </visual>
+    <collision>
+      <origin xyz="0 0 0" rpy="0 0 0"/>
+      <geometry>
+        <mesh filename="file://$(find summit_xl_description)/meshes/structures/d455_base.stl" scale="0.001 0.001 0.001"/>
+      </geometry>
+    </collision>
+  </link>
+  <joint name="$(arg prefix)/d455_base_joint" type="fixed">
+    <origin rpy="-${pi/2} 0.0 ${pi/2}" xyz="0.0105 0.0 0.243"/>
+    <parent link="$(arg prefix)/camera_mast_link" />
+    <child link="$(arg prefix)/d455_base_link" />
+  </joint>
+  <xacro:sensor_d455 parent="$(arg prefix)/d455_base_link" use_nominal_extrinsics="true">
+    <origin xyz="0.0 0.017 -0.005" rpy="0 ${pi-pi/3} -${pi/2}"/>
+  </xacro:sensor_d455>
   <!-- GPS -->
   <xacro:structure_mastil_gps prefix="$(arg prefix)/gps" parent="$(arg prefix)/base_link">
